File: JuxtaN1.kicad_sch (KiCad schematic)
At the start: 18 parts, among them IC1 BGM220SC12WGA2R, J1 Conn_02x05_Odd_Even, U1 TPS61099x_YFF, U2 Si7210-B-xx-IM2, U3 LSM6DS3, Y1 Crystal

Commit message: Considering other AFEs
Parts:
- removed U4: ~, JuxtaN:BGA-36_6x6_2.6x2.5mm, symbol JuxtaN_SchematicLib:AFE4950
- added IC2: MAX30003CWV+T, BGA30C50P6X5_293X274X69, symbol MAX30003:MAX30003CWV+T
